Commit message: 1.0.1

File: urdf/robot.urdf (robot description, URDF)
Before this commit: robot botAlive, 1 links, 0 joints
Links:
- removed link chassis
- added link link_arm, mass 1; collision box size=0.2 0.2 1; visual box size=0.2 0.2 1
- added link link_chassis, mass 3.07549; collision box size=2 2 1; visual box size=2 2 1
Joints:
- added joint joint1: type continuous, parent link_chassis, child link_arm, origin xyz=0.6 0 0.5 rpy=0 0 0

Commit message: 1.0.2

File: urdf/robot.urdf (robot description, URDF)
Before this commit: robot botAlive, 2 links, 1 joints
Links:
- removed link link_arm
- removed link link_chassis
- added link base_link, mass 3.07549; collision box size=0.18 0.12 0.06; visual box size=0.18 0.12 0.06
- added link lwheel; visual cylinder length=0.012 radius=0.06
- added link rwheel; visual cylinder length=0.012 radius=0.06
- added link scanner; visual box size=0.015 0.045 0.025
Joints:
- removed joint joint1
- added joint base_to_lwheel: type fixed, parent base_link, child lwheel, origin xyz=0 0.075 0.046 rpy=1.5708 0 0
- added joint base_to_rwheel: type fixed, parent base_link, child rwheel, origin xyz=0 -0.075 0.046 rpy=-1.5708 0 0
- added joint base_to_scanner: type fixed, parent base_link, child scanner, origin xyz=0.105 0 0.06 rpy=0 0 0
